File: trabajoProfesional/Bateria.sch (KiCad schematic (older format))
At the start: 26 parts

Commit message: ya tenemos los componentes falta el micro
Parts:
- removed Cs1: C, symbol Device:C
- Cbat, Cvin: value C -> 2.2u
- Cbst: value C -> 47n
- Cc1, Cc2: value C -> 1n
- Cin1, Cout1, Cout2, Cout3, Cout4: value C -> 22u
- Cin2: value C -> 100n
- Cs2: value C -> 10n
- Lout: value L -> 4.7u
- R1fb: renamed from R?; value R -> 46k
- R2fb: renamed from R?; value R -> 10k
- Rmod_cfg: value R -> 60k
- gave numbers to parts that had none: 1
Changed lines of the file:
@@
 P 1750 2200
 F 0 "Cs2" V 1498 2200 50  0000 C CNN
-F 1 "C" V 1589 2200 50  0000 C CNN
+F 1 "10n" V 1589 2200 50  0000 C CNN
 F 2 "" H 1788 2050 50  0001 C CNN
 F 3 "~" H 1750 2200 50  0001 C CNN
@@
 P 1550 3100
 F 0 "Cc1" H 1435 3054 50  0000 R CNN
-F 1 "C" H 1435 3145 50  0000 R CNN
+F 1 "1n" H 1435 3145 50  0000 R CNN
 F 2 "" H 1588 2950 50  0001 C CNN
 F 3 "~" H 1550 3100 50  0001 C CNN
@@
 P 2950 2400
 F 0 "Cc2" V 3202 2400 50  0000 C CNN
-F 1 "C" V 3111 2400 50  0000 C CNN
+F 1 "1n" V 3111 2400 50  0000 C CNN
 F 2 "" H 2988 2250 50  0001 C CNN
 F 3 "~" H 2950 2400 50  0001 C CNN
@@
 P 2300 3050
 F 0 "Cbst" H 2185 3004 50  0000 R CNN
-F 1 "C" H 2185 3095 50  0000 R CNN
+F 1 "47n" H 2185 3095 50  0000 R CNN
 F 2 "" H 2338 2900 50  0001 C CNN
 F 3 "~" H 2300 3050 50  0001 C CNN
@@
 P 5300 2350
 F 0 "Cin1" H 5185 2304 50  0000 R CNN
-F 1 "C" H 5185 2395 50  0000 R CNN
+F 1 "22u" H 5185 2395 50  0000 R CNN
 F 2 "" H 5338 2200 50  0001 C CNN
 F 3 "~" H 5300 2350 50  0001 C CNN
@@
 P 7000 2500
 F 0 "Lout" V 6819 2500 50  0000 C CNN
-F 1 "L" V 6910 2500 50  0000 C CNN
+F 1 "4.7u" V 6910 2500 50  0000 C CNN
 F 2 "" H 7000 2500 50  0001 C CNN
 F 3 "~" H 7000 2500 50  0001 C CNN
@@
 P 5550 2900
 F 0 "Rmod_cfg" H 5620 2946 50  0000 L CNN
-F 1 "R" H 5620 2855 50  0000 L CNN
+F 1 "60k" H 5620 2855 50  0000 L CNN
 F 2 "" V 5480 2900 50  0001 C CNN
 F 3 "~" H 5550 2900 50  0001 C CNN
@@
 $EndComp
 Wire Wire Line
-	1600 2200 1450 2200
-Wire Wire Line
 	1300 2200 1300 2250
 Wire Wire Line
@@
 Wire Wire Line
 	1550 2550 2700 2550
-Wire Wire Line
-	1900 2200 2050 2200
 Wire Wire Line
 	3100 2400 3300 2400
@@
 Connection ~ 3300 3250
 $Comp
-L Device:C Cs1
-U 1 1 5F3FF8AC
-P 1750 1800
-F 0 "Cs1" V 1498 1800 50  0000 C CNN
-F 1 "C" V 1589 1800 50  0000 C CNN
-F 2 "" H 1788 1650 50  0001 C CNN
-F 3 "~" H 1750 1800 50  0001 C CNN
-	1    1750 1800
-	0    1    1    0
-$EndComp
-Wire Wire Line
-	1900 1800 2050 1800
-Wire Wire Line
-	2050 1800 2050 2200
-Connection ~ 2050 2200
-Wire Wire Line
-	2050 2200 2800 2200
-Wire Wire Line
-	1450 2200 1450 1800
-Wire Wire Line
-	1450 1800 1600 1800
-Connection ~ 1450 2200
-Wire Wire Line
-	1450 2200 1300 2200
-$Comp
 L Device:C Cin2
 U 1 1 5F40192A
 P 5700 2350
 F 0 "Cin2" H 5585 2304 50  0000 R CNN
-F 1 "C" H 5585 2395 50  0000 R CNN
+F 1 "100n" H 5585 2395 50  0000 R CNN
 F 2 "" H 5738 2200 50  0001 C CNN
 F 3 "~" H 5700 2350 50  0001 C CNN
@@
 Connection ~ 4700 2200
 $Comp
-L Device:R R?
+L Device:R R1fb
 U 1 1 5F4084FD
 P 7300 2650
-F 0 "R?" H 7370 2696 50  0000 L CNN
-F 1 "R" H 7370 2605 50  0000 L CNN
+F 0 "R1fb" H 7370 2696 50  0000 L CNN
+F 1 "46k" H 7370 2605 50  0000 L CNN
 F 2 "" V 7230 2650 50  0001 C CNN
 F 3 "~" H 7300 2650 50  0001 C CNN
@@
 $EndComp
 $Comp
-L Device:R R?
+L Device:R R2fb
 U 1 1 5F408C04
 P 7300 3050
-F 0 "R?" H 7230 3004 50  0000 R CNN
-F 1 "R" H 7230 3095 50  0000 R CNN
+F 0 "R2fb" H 7230 3004 50  0000 R CNN
+F 1 "10k" H 7230 3095 50  0000 R CNN
 F 2 "" V 7230 3050 50  0001 C CNN
 F 3 "~" H 7300 3050 50  0001 C CNN
@@
 P 7650 2650
 F 0 "Cout1" H 7535 2604 50  0000 R CNN
-F 1 "C" H 7535 2695 50  0000 R CNN
+F 1 "22u" H 7535 2695 50  0000 R CNN
 F 2 "" H 7688 2500 50  0001 C CNN
 F 3 "~" H 7650 2650 50  0001 C CNN
@@
 P 8050 2650
 F 0 "Cout2" H 7935 2604 50  0000 R CNN
-F 1 "C" H 7935 2695 50  0000 R CNN
+F 1 "22u" H 7935 2695 50  0000 R CNN
 F 2 "" H 8088 2500 50  0001 C CNN
 F 3 "~" H 8050 2650 50  0001 C CNN
@@
 P 8450 2650
 F 0 "Cout3" H 8335 2604 50  0000 R CNN
-F 1 "C" H 8335 2695 50  0000 R CNN
+F 1 "22u" H 8335 2695 50  0000 R CNN
 F 2 "" H 8488 2500 50  0001 C CNN
 F 3 "~" H 8450 2650 50  0001 C CNN
@@
 P 8750 2650
 F 0 "Cout4" H 8635 2604 50  0000 R CNN
-F 1 "C" H 8635 2695 50  0000 R CNN
+F 1 "22u" H 8635 2695 50  0000 R CNN
 F 2 "" H 8788 2500 50  0001 C CNN
 F 3 "~" H 8750 2650 50  0001 C CNN
@@
 P 6150 5250
 F 0 "Cbat" H 6265 5296 50  0000 L CNN
-F 1 "C" H 6265 5205 50  0000 L CNN
+F 1 "2.2u" H 6265 5205 50  0000 L CNN
 F 2 "" H 6188 5100 50  0001 C CNN
 F 3 "~" H 6150 5250 50  0001 C CNN
@@
 Connection ~ 6150 5050
 $Comp
-L pspice:MPMOS M?
+L pspice:MPMOS T1
 U 1 1 5F4412C3
 P 7200 4750
-F 0 "M?" H 7488 4796 50  0000 L CNN
+F 0 "T1" H 7488 4796 50  0000 L CNN
 F 1 "MPMOS" H 7488 4705 50  0000 L CNN
 F 2 "" H 7200 4750 50  0001 C CNN
@@
 P 3100 4750
 F 0 "Cvin" V 2848 4750 50  0000 C CNN
-F 1 "C" V 2939 4750 50  0000 C CNN
+F 1 "2.2u" V 2939 4750 50  0000 C CNN
 F 2 "" H 3138 4600 50  0001 C CNN
 F 3 "~" H 3100 4750 50  0001 C CNN
@@
 	3300 5050 3350 5050
 Connection ~ 3350 5050
+Wire Wire Line
+	1300 2200 1600 2200
+Wire Wire Line
+	1900 2200 2800 2200
 $EndSCHEMATC

Commit message: empezando el pcb
Parts:
- AdministracionBateria1: renamed from AdministracionBateria; footprint SON50P200X200X60-7N-D -> SC810:SON50P200X200X60-7N-D
- Cbat1: renamed from Cbat; footprint (none) -> Capacitor_SMD:C_Elec_3x5.4
- Cbst1: renamed from Cbst; footprint (none) -> Capacitor_SMD:C_2816_7142Metric
- Cc1, Cc2, Cin1, Cin2, Cout1, Cout2, Cout3, Cout4, Cs2: footprint (none) -> Capacitor_SMD:CP_Elec_3x5.3
- Cvin1: renamed from Cvin; footprint (none) -> Capacitor_SMD:C_Elec_3x5.4
- DbyPass1: renamed from DbyPass; footprint (none) -> Diode_SMD:D_SOD-323F
- Lout1: renamed from Lout; footprint (none) -> Inductor_SMD:L_7.3x7.3_H3.5
- R1fb1: renamed from R1fb; footprint (none) -> Resistor_SMD:R_1206_3216Metric
- R2fb1: renamed from R2fb; footprint (none) -> Resistor_SMD:R_1206_3216Metric
- RIPRGM1: renamed from RIPRGM; footprint (none) -> Resistor_SMD:R_1206_3216Metric
- RecpetorPotenciaInalambrica1: renamed from RecpetorPotenciaInalambrica; footprint BGA20C40P4X5_190X230X58 -> TS51223:BGA20C40P4X5_190X230X58
- Riso_pd1: renamed from Riso_pd; footprint (none) -> Resistor_SMD:R_1206_3216Metric
- Rmod_cfg1: renamed from Rmod_cfg; footprint (none) -> Resistor_SMD:R_1206_3216Metric
- Rstatus1: renamed from Rstatus; footprint (none) -> Resistor_SMD:R_1206_3216Metric
- T1: footprint (none) -> Package_TO_SOT_SMD:TSOT-23
- coil1: renamed from coil; footprint (none) -> Connector_PinHeader_2.54mm:PinHeader_1x02_P2.54mm_Vertical
- opt1: renamed from opt; footprint (none) -> Diode_SMD:D_SOD-323F
Changed lines of the file:
@@
 $EndDescr
 $Comp
-L TS51223-M000WCSR:TS51223-M000WCSR RecpetorPotenciaInalambrica
+L TS51223-M000WCSR:TS51223-M000WCSR RecpetorPotenciaInalambrica1
 U 1 1 5F3EC0E0
 P 3300 2200
-F 0 "RecpetorPotenciaInalambrica" H 4000 2465 50  0000 C CNN
+F 0 "RecpetorPotenciaInalambrica1" H 4000 2465 50  0000 C CNN
 F 1 "TS51223-M000WCSR" H 4000 2374 50  0000 C CNN
-F 2 "BGA20C40P4X5_190X230X58" H 4550 2300 50  0001 L CNN
+F 2 "TS51223:BGA20C40P4X5_190X230X58" H 4550 2300 50  0001 L CNN
 F 3 "https://componentsearchengine.com/Datasheets/1/TS51223-M000WCSR.pdf" H 4550 2200 50  0001 L CNN
 F 4 "Wireless Charging ICs Wireless Port Rec. Ext Resistor Fbk" H 4550 2100 50  0001 L CNN "Description"
@@
 $EndComp
 $Comp
-L SC810ULTRT:SC810ULTRT AdministracionBateria
+L SC810ULTRT:SC810ULTRT AdministracionBateria1
 U 1 1 5F3EDAD5
 P 3500 4950
-F 0 "AdministracionBateria" H 4100 5215 50  0000 C CNN
+F 0 "AdministracionBateria1" H 4100 5215 50  0000 C CNN
 F 1 "SC810ULTRT" H 4100 5124 50  0000 C CNN
-F 2 "SON50P200X200X60-7N-D" H 4550 5050 50  0001 L CNN
+F 2 "SC810:SON50P200X200X60-7N-D" H 4550 5050 50  0001 L CNN
 F 3 "https://www.arrow.com/en/products/sc810ultrt/semtech" H 4550 4950 50  0001 L CNN
 F 4 "Battery Management SNGL INPUT/MODE LI BATT CHRGR" H 4550 4850 50  0001 L CNN "Description"
@@
 $EndComp
 $Comp
-L Device:L coil
+L Device:L coil1
 U 1 1 5F3EE7F6
 P 1300 2400
-F 0 "coil" H 1352 2446 50  0000 L CNN
+F 0 "coil1" H 1352 2446 50  0000 L CNN
 F 1 "L" H 1352 2355 50  0000 L CNN
-F 2 "" H 1300 2400 50  0001 C CNN
+F 2 "Connector_PinHeader_2.54mm:PinHeader_1x02_P2.54mm_Vertical" H 1300 2400 50  0001 C CNN
 F 3 "~" H 1300 2400 50  0001 C CNN
 	1    1300 2400
@@
 F 0 "Cs2" V 1498 2200 50  0000 C CNN
 F 1 "10n" V 1589 2200 50  0000 C CNN
-F 2 "" H 1788 2050 50  0001 C CNN
+F 2 "Capacitor_SMD:CP_Elec_3x5.3" H 1788 2050 50  0001 C CNN
 F 3 "~" H 1750 2200 50  0001 C CNN
 	1    1750 2200
@@
 F 0 "Cc1" H 1435 3054 50  0000 R CNN
 F 1 "1n" H 1435 3145 50  0000 R CNN
-F 2 "" H 1588 2950 50  0001 C CNN
+F 2 "Capacitor_SMD:CP_Elec_3x5.3" H 1588 2950 50  0001 C CNN
 F 3 "~" H 1550 3100 50  0001 C CNN
 	1    1550 3100
@@
 F 0 "Cc2" V 3202 2400 50  0000 C CNN
 F 1 "1n" V 3111 2400 50  0000 C CNN
-F 2 "" H 2988 2250 50  0001 C CNN
+F 2 "Capacitor_SMD:CP_Elec_3x5.3" H 2988 2250 50  0001 C CNN
 F 3 "~" H 2950 2400 50  0001 C CNN
 	1    2950 2400
@@
 $EndComp
 $Comp
-L Device:C Cbst
+L Device:C Cbst1
 U 1 1 5F3F119B
 P 2300 3050
-F 0 "Cbst" H 2185 3004 50  0000 R CNN
+F 0 "Cbst1" H 2185 3004 50  0000 R CNN
 F 1 "47n" H 2185 3095 50  0000 R CNN
-F 2 "" H 2338 2900 50  0001 C CNN
+F 2 "Capacitor_SMD:C_2816_7142Metric" H 2338 2900 50  0001 C CNN
 F 3 "~" H 2300 3050 50  0001 C CNN
 	1    2300 3050
@@
 F 0 "Cin1" H 5185 2304 50  0000 R CNN
 F 1 "22u" H 5185 2395 50  0000 R CNN
-F 2 "" H 5338 2200 50  0001 C CNN
+F 2 "Capacitor_SMD:CP_Elec_3x5.3" H 5338 2200 50  0001 C CNN
 F 3 "~" H 5300 2350 50  0001 C CNN
 	1    5300 2350
@@
 $EndComp
 $Comp
-L Device:L Lout
+L Device:L Lout1
 U 1 1 5F3F1D24
 P 7000 2500
-F 0 "Lout" V 6819 2500 50  0000 C CNN
+F 0 "Lout1" V 6819 2500 50  0000 C CNN
 F 1 "4.7u" V 6910 2500 50  0000 C CNN
-F 2 "" H 7000 2500 50  0001 C CNN
+F 2 "Inductor_SMD:L_7.3x7.3_H3.5" H 7000 2500 50  0001 C CNN
 F 3 "~" H 7000 2500 50  0001 C CNN
 	1    7000 2500
@@
 $EndComp
 $Comp
-L Device:R Rmod_cfg
+L Device:R Rmod_cfg1
 U 1 1 5F3F2621
 P 5550 2900
-F 0 "Rmod_cfg" H 5620 2946 50  0000 L CNN
+F 0 "Rmod_cfg1" H 5620 2946 50  0000 L CNN
 F 1 "60k" H 5620 2855 50  0000 L CNN
-F 2 "" V 5480 2900 50  0001 C CNN
+F 2 "Resistor_SMD:R_1206_3216Metric" V 5480 2900 50  0001 C CNN
 F 3 "~" H 5550 2900 50  0001 C CNN
 	1    5550 2900
@@
 	1550 3500 1550 3250
 $Comp
-L power:GND #PWR?
+L power:GND #PWR0103
 U 1 1 5F3F635E
 P 2600 2650
-F 0 "#PWR?" H 2600 2400 50  0001 C CNN
+F 0 "#PWR0103" H 2600 2400 50  0001 C CNN
 F 1 "GND" H 2605 2477 50  0000 C CNN
 F 2 "" H 2600 2650 50  0001 C CNN
@@
 F 0 "Cin2" H 5585 2304 50  0000 R CNN
 F 1 "100n" H 5585 2395 50  0000 R CNN
-F 2 "" H 5738 2200 50  0001 C CNN
+F 2 "Capacitor_SMD:CP_Elec_3x5.3" H 5738 2200 50  0001 C CNN
 F 3 "~" H 5700 2350 50  0001 C CNN
 	1    5700 2350
@@
 Connection ~ 4700 2200
 $Comp
-L Device:R R1fb
+L Device:R R1fb1
 U 1 1 5F4084FD
 P 7300 2650
-F 0 "R1fb" H 7370 2696 50  0000 L CNN
+F 0 "R1fb1" H 7370 2696 50  0000 L CNN
 F 1 "46k" H 7370 2605 50  0000 L CNN
-F 2 "" V 7230 2650 50  0001 C CNN
+F 2 "Resistor_SMD:R_1206_3216Metric" V 7230 2650 50  0001 C CNN
 F 3 "~" H 7300 2650 50  0001 C CNN
 	1    7300 2650
@@
 $EndComp
 $Comp
-L Device:R R2fb
+L Device:R R2fb1
 U 1 1 5F408C04
 P 7300 3050
-F 0 "R2fb" H 7230 3004 50  0000 R CNN
+F 0 "R2fb1" H 7230 3004 50  0000 R CNN
 F 1 "10k" H 7230 3095 50  0000 R CNN
-F 2 "" V 7230 3050 50  0001 C CNN
+F 2 "Resistor_SMD:R_1206_3216Metric" V 7230 3050 50  0001 C CNN
 F 3 "~" H 7300 3050 50  0001 C CNN
 	1    7300 3050
@@
 F 0 "Cout1" H 7535 2604 50  0000 R CNN
 F 1 "22u" H 7535 2695 50  0000 R CNN
-F 2 "" H 7688 2500 50  0001 C CNN
+F 2 "Capacitor_SMD:CP_Elec_3x5.3" H 7688 2500 50  0001 C CNN
 F 3 "~" H 7650 2650 50  0001 C CNN
 	1    7650 2650
@@
 F 0 "Cout2" H 7935 2604 50  0000 R CNN
 F 1 "22u" H 7935 2695 50  0000 R CNN
-F 2 "" H 8088 2500 50  0001 C CNN
+F 2 "Capacitor_SMD:CP_Elec_3x5.3" H 8088 2500 50  0001 C CNN
 F 3 "~" H 8050 2650 50  0001 C CNN
 	1    8050 2650
@@
 F 0 "Cout3" H 8335 2604 50  0000 R CNN
 F 1 "22u" H 8335 2695 50  0000 R CNN
-F 2 "" H 8488 2500 50  0001 C CNN
+F 2 "Capacitor_SMD:CP_Elec_3x5.3" H 8488 2500 50  0001 C CNN
 F 3 "~" H 8450 2650 50  0001 C CNN
 	1    8450 2650
@@
 F 0 "Cout4" H 8635 2604 50  0000 R CNN
 F 1 "22u" H 8635 2695 50  0000 R CNN
-F 2 "" H 8788 2500 50  0001 C CNN
+F 2 "Capacitor_SMD:CP_Elec_3x5.3" H 8788 2500 50  0001 C CNN
 F 3 "~" H 8750 2650 50  0001 C CNN
 	1    8750 2650
@@
 	2850 3350 2850 4750
 $Comp
-L Device:R RIPRGM
+L Device:R RIPRGM1
 U 1 1 5F427DAE
 P 5100 5200
-F 0 "RIPRGM" V 4893 5200 50  0000 C CNN
+F 0 "RIPRGM1" V 4893 5200 50  0000 C CNN
 F 1 "R" V 4984 5200 50  0000 C CNN
-F 2 "" V 5030 5200 50  0001 C CNN
+F 2 "Resistor_SMD:R_1206_3216Metric" V 5030 5200 50  0001 C CNN
 F 3 "~" H 5100 5200 50  0001 C CNN
 	1    5100 5200
@@
 Connection ~ 5250 5200
 $Comp
-L Device:C Cbat
+L Device:C Cbat1
 U 1 1 5F42FDFF
 P 6150 5250
-F 0 "Cbat" H 6265 5296 50  0000 L CNN
+F 0 "Cbat1" H 6265 5296 50  0000 L CNN
 F 1 "2.2u" H 6265 5205 50  0000 L CNN
-F 2 "" H 6188 5100 50  0001 C CNN
+F 2 "Capacitor_SMD:C_Elec_3x5.4" H 6188 5100 50  0001 C CNN
 F 3 "~" H 6150 5250 50  0001 C CNN
 	1    6150 5250
@@
 F 0 "T1" H 7488 4796 50  0000 L CNN
 F 1 "MPMOS" H 7488 4705 50  0000 L CNN
-F 2 "" H 7200 4750 50  0001 C CNN
+F 2 "Package_TO_SOT_SMD:TSOT-23" H 7200 4750 50  0001 C CNN
 F 3 "~" H 7200 4750 50  0001 C CNN
 	1    7200 4750
@@
 Connection ~ 7300 4550
 $Comp
-L Device:R Riso_pd
+L Device:R Riso_pd1
 U 1 1 5F44B6C8
 P 6400 4700
-F 0 "Riso_pd" H 6330 4654 50  0000 R CNN
+F 0 "Riso_pd1" H 6330 4654 50  0000 R CNN
 F 1 "R" H 6330 4745 50  0000 R CNN
-F 2 "" V 6330 4700 50  0001 C CNN
+F 2 "Resistor_SMD:R_1206_3216Metric" V 6330 4700 50  0001 C CNN
 F 3 "~" H 6400 4700 50  0001 C CNN
 	1    6400 4700
@@
 	6400 3700 10000 3700
 $Comp
-L Device:C Cvin
+L Device:C Cvin1
 U 1 1 5F456249
 P 3100 4750
-F 0 "Cvin" V 2848 4750 50  0000 C CNN
+F 0 "Cvin1" V 2848 4750 50  0000 C CNN
 F 1 "2.2u" V 2939 4750 50  0000 C CNN
-F 2 "" H 3138 4600 50  0001 C CNN
+F 2 "Capacitor_SMD:C_Elec_3x5.4" H 3138 4600 50  0001 C CNN
 F 3 "~" H 3100 4750 50  0001 C CNN
 	1    3100 4750
@@
 	2850 4750 2850 5150
 $Comp
-L Device:D_Schottky opt
+L Device:D_Schottky opt1
 U 1 1 5F466CB6
 P 5700 4600
-F 0 "opt" V 5654 4680 50  0000 L CNN
+F 0 "opt1" V 5654 4680 50  0000 L CNN
 F 1 "D_Schottky" V 5745 4680 50  0000 L CNN
-F 2 "" H 5700 4600 50  0001 C CNN
+F 2 "Diode_SMD:D_SOD-323F" H 5700 4600 50  0001 C CNN
 F 3 "~" H 5700 4600 50  0001 C CNN
 	1    5700 4600
@@
 $EndComp
 $Comp
-L Device:D_Schottky DbyPass
+L Device:D_Schottky DbyPass1
 U 1 1 5F467739
 P 5300 4050
-F 0 "DbyPass" H 5300 3833 50  0000 C CNN
+F 0 "DbyPass1" H 5300 3833 50  0000 C CNN
 F 1 "D_Schottky" H 5300 3924 50  0000 C CNN
-F 2 "" H 5300 4050 50  0001 C CNN
+F 2 "Diode_SMD:D_SOD-323F" H 5300 4050 50  0001 C CNN
 F 3 "~" H 5300 4050 50  0001 C CNN
 	1    5300 4050
@@
 	3500 4050 3500 4750
 $Comp
-L Device:R Rstatus
+L Device:R Rstatus1
 U 1 1 5F478013
 P 4050 4500
-F 0 "Rstatus" V 3843 4500 50  0000 C CNN
+F 0 "Rstatus1" V 3843 4500 50  0000 C CNN
 F 1 "R" V 3934 4500 50  0000 C CNN
-F 2 "" V 3980 4500 50  0001 C CNN
+F 2 "Resistor_SMD:R_1206_3216Metric" V 3980 4500 50  0001 C CNN
 F 3 "~" H 4050 4500 50  0001 C CNN
 	1    4050 4500

Commit message: paso previo PCB
Parts:
- removed coil1: L, Connector_PinHeader_2.54mm:PinHeader_1x02_P2.54mm_Vertical, symbol Device:L
- added BatPositivo1, Coil1, Coil2, batGND1: Conn_01x01_Male, Connector_PinHeader_1.00mm:PinHeader_1x01_P1.00mm_Vertical, symbol Connector:Conn_01x01_Male
Connections:
- net +Bat: now also BatPositivo1.1 (Pin_1)
- net GND: now also batGND1.1 (Pin_1)
- net at Cc1.2, RecpetorPotenciaInalambrica1.E1 (VAC2): now also Coil2.1 (Pin_1)
- net at Cs2.2: now also Coil1.1 (Pin_1)
Changed lines of the file:
@@
-$EndComp
-$Comp
-L Device:L coil1
-U 1 1 5F3EE7F6
-P 1300 2400
-F 0 "coil1" H 1352 2446 50  0000 L CNN
-F 1 "L" H 1352 2355 50  0000 L CNN
-F 2 "Connector_PinHeader_2.54mm:PinHeader_1x02_P2.54mm_Vertical" H 1300 2400 50  0001 C CNN
-F 3 "~" H 1300 2400 50  0001 C CNN
-	1    1300 2400
-	1    0    0    -1
 $EndComp
 $Comp
@@
 $EndComp
 Wire Wire Line
-	1300 2200 1300 2250
-Wire Wire Line
 	2700 2550 2700 1650
 Wire Wire Line
@@
 Wire Wire Line
 	5000 2800 4700 2800
-Wire Wire Line
-	1300 2550 1550 2550
 Wire Wire Line
 	1550 2950 1550 2550
@@
 +Bat
 Wire Wire Line
-	7300 5250 7300 5050
-Wire Wire Line
 	7300 5050 6150 5050
 Connection ~ 6150 5050
@@
 Connection ~ 3350 5050
 Wire Wire Line
-	1300 2200 1600 2200
-Wire Wire Line
 	1900 2200 2800 2200
+Wire Wire Line
+	7300 5050 7300 5550
+$Comp
+L power:GND #PWR0104
+U 1 1 5F3F986E
+P 7300 5850
+F 0 "#PWR0104" H 7300 5600 50  0001 C CNN
+F 1 "GND" H 7305 5677 50  0000 C CNN
+F 2 "" H 7300 5850 50  0001 C CNN
+F 3 "" H 7300 5850 50  0001 C CNN
+	1    7300 5850
+	1    0    0    -1
+$EndComp
+Wire Wire Line
+	7300 5650 7300 5850
+$Comp
+L Connector:Conn_01x01_Male Coil1
+U 1 1 5F4171CB
+P 1050 2200
+F 0 "Coil1" H 1158 2381 50  0000 C CNN
+F 1 "Conn_01x01_Male" H 1158 2290 50  0000 C CNN
+F 2 "Connector_PinHeader_1.00mm:PinHeader_1x01_P1.00mm_Vertical" H 1050 2200 50  0001 C CNN
+F 3 "~" H 1050 2200 50  0001 C CNN
+	1    1050 2200
+	1    0    0    -1
+$EndComp
+$Comp
+L Connector:Conn_01x01_Male Coil2
+U 1 1 5F417846
+P 1050 2550
+F 0 "Coil2" H 1158 2731 50  0000 C CNN
+F 1 "Conn_01x01_Male" H 1158 2640 50  0000 C CNN
+F 2 "Connector_PinHeader_1.00mm:PinHeader_1x01_P1.00mm_Vertical" H 1050 2550 50  0001 C CNN
+F 3 "~" H 1050 2550 50  0001 C CNN
+	1    1050 2550
+	1    0    0    -1
+$EndComp
+Wire Wire Line
+	1250 2200 1600 2200
+Wire Wire Line
+	1250 2550 1550 2550
+$Comp
+L Connector:Conn_01x01_Male BatPositivo1
+U 1 1 5F421506
+P 7800 5550
+F 0 "BatPositivo1" H 7772 5482 50  0000 R CNN
+F 1 "Conn_01x01_Male" H 7772 5573 50  0000 R CNN
+F 2 "Connector_PinHeader_1.00mm:PinHeader_1x01_P1.00mm_Vertical" H 7800 5550 50  0001 C CNN
+F 3 "~" H 7800 5550 50  0001 C CNN
+	1    7800 5550
+	-1   0    0    1
+$EndComp
+$Comp
+L Connector:Conn_01x01_Male batGND1
+U 1 1 5F421C96
+P 6750 5650
+F 0 "batGND1" H 6858 5831 50  0000 C CNN
+F 1 "Conn_01x01_Male" H 6858 5740 50  0000 C CNN
+F 2 "Connector_PinHeader_1.00mm:PinHeader_1x01_P1.00mm_Vertical" H 6750 5650 50  0001 C CNN
+F 3 "~" H 6750 5650 50  0001 C CNN
+	1    6750 5650
+	1    0    0    -1
+$EndComp
+Wire Wire Line
+	7600 5550 7300 5550
+Wire Wire Line
+	7300 5650 6950 5650
 $EndSCHEMATC

Commit message: PCB falta una conexion
Parts:
- BatPositivo1, Coil1, Coil2, batGND1: footprint Connector_PinHeader_1.00mm:PinHeader_1x01_P1.00mm_Vertical -> TestPoint:TestPoint_Pad_D2.5mm
Changed lines of the file:
@@
 F 0 "Coil1" H 1158 2381 50  0000 C CNN
 F 1 "Conn_01x01_Male" H 1158 2290 50  0000 C CNN
-F 2 "Connector_PinHeader_1.00mm:PinHeader_1x01_P1.00mm_Vertical" H 1050 2200 50  0001 C CNN
+F 2 "TestPoint:TestPoint_Pad_D2.5mm" H 1050 2200 50  0001 C CNN
 F 3 "~" H 1050 2200 50  0001 C CNN
 	1    1050 2200
@@
 F 0 "Coil2" H 1158 2731 50  0000 C CNN
 F 1 "Conn_01x01_Male" H 1158 2640 50  0000 C CNN
-F 2 "Connector_PinHeader_1.00mm:PinHeader_1x01_P1.00mm_Vertical" H 1050 2550 50  0001 C CNN
+F 2 "TestPoint:TestPoint_Pad_D2.5mm" H 1050 2550 50  0001 C CNN
 F 3 "~" H 1050 2550 50  0001 C CNN
 	1    1050 2550
@@
 F 0 "BatPositivo1" H 7772 5482 50  0000 R CNN
 F 1 "Conn_01x01_Male" H 7772 5573 50  0000 R CNN
-F 2 "Connector_PinHeader_1.00mm:PinHeader_1x01_P1.00mm_Vertical" H 7800 5550 50  0001 C CNN
+F 2 "TestPoint:TestPoint_Pad_D2.5mm" H 7800 5550 50  0001 C CNN
 F 3 "~" H 7800 5550 50  0001 C CNN
 	1    7800 5550
@@
 F 0 "batGND1" H 6858 5831 50  0000 C CNN
 F 1 "Conn_01x01_Male" H 6858 5740 50  0000 C CNN
-F 2 "Connector_PinHeader_1.00mm:PinHeader_1x01_P1.00mm_Vertical" H 6750 5650 50  0001 C CNN
+F 2 "TestPoint:TestPoint_Pad_D2.5mm" H 6750 5650 50  0001 C CNN
 F 3 "~" H 6750 5650 50  0001 C CNN
 	1    6750 5650

Commit message: va el circuito
Parts:
- Cbst1: footprint Capacitor_SMD:C_2816_7142Metric -> Capacitor_SMD:C_0201_0603Metric
- R1fb1, R2fb1, RIPRGM1, Riso_pd1, Rmod_cfg1: footprint Resistor_SMD:R_1206_3216Metric -> Resistor_SMD:R_0201_0603Metric
- Rstatus1: footprint Resistor_SMD:R_1206_3216Metric -> Resistor_SMD:R_1806_4516Metric
Changed lines of the file:
@@
 F 0 "Cbst1" H 2185 3004 50  0000 R CNN
 F 1 "47n" H 2185 3095 50  0000 R CNN
-F 2 "Capacitor_SMD:C_2816_7142Metric" H 2338 2900 50  0001 C CNN
+F 2 "Capacitor_SMD:C_0201_0603Metric" H 2338 2900 50  0001 C CNN
 F 3 "~" H 2300 3050 50  0001 C CNN
 	1    2300 3050
@@
 F 0 "Rmod_cfg1" H 5620 2946 50  0000 L CNN
 F 1 "60k" H 5620 2855 50  0000 L CNN
-F 2 "Resistor_SMD:R_1206_3216Metric" V 5480 2900 50  0001 C CNN
+F 2 "Resistor_SMD:R_0201_0603Metric" V 5480 2900 50  0001 C CNN
 F 3 "~" H 5550 2900 50  0001 C CNN
 	1    5550 2900
@@
 F 0 "R1fb1" H 7370 2696 50  0000 L CNN
 F 1 "46k" H 7370 2605 50  0000 L CNN
-F 2 "Resistor_SMD:R_1206_3216Metric" V 7230 2650 50  0001 C CNN
+F 2 "Resistor_SMD:R_0201_0603Metric" V 7230 2650 50  0001 C CNN
 F 3 "~" H 7300 2650 50  0001 C CNN
 	1    7300 2650
@@
 F 0 "R2fb1" H 7230 3004 50  0000 R CNN
 F 1 "10k" H 7230 3095 50  0000 R CNN
-F 2 "Resistor_SMD:R_1206_3216Metric" V 7230 3050 50  0001 C CNN
+F 2 "Resistor_SMD:R_0201_0603Metric" V 7230 3050 50  0001 C CNN
 F 3 "~" H 7300 3050 50  0001 C CNN
 	1    7300 3050
@@
 F 0 "RIPRGM1" V 4893 5200 50  0000 C CNN
 F 1 "R" V 4984 5200 50  0000 C CNN
-F 2 "Resistor_SMD:R_1206_3216Metric" V 5030 5200 50  0001 C CNN
+F 2 "Resistor_SMD:R_0201_0603Metric" V 5030 5200 50  0001 C CNN
 F 3 "~" H 5100 5200 50  0001 C CNN
 	1    5100 5200
@@
 F 0 "Riso_pd1" H 6330 4654 50  0000 R CNN
 F 1 "R" H 6330 4745 50  0000 R CNN
-F 2 "Resistor_SMD:R_1206_3216Metric" V 6330 4700 50  0001 C CNN
+F 2 "Resistor_SMD:R_0201_0603Metric" V 6330 4700 50  0001 C CNN
 F 3 "~" H 6400 4700 50  0001 C CNN
 	1    6400 4700
@@
 F 0 "Rstatus1" V 3843 4500 50  0000 C CNN
 F 1 "R" V 3934 4500 50  0000 C CNN
-F 2 "Resistor_SMD:R_1206_3216Metric" V 3980 4500 50  0001 C CNN
+F 2 "Resistor_SMD:R_1806_4516Metric" V 3980 4500 50  0001 C CNN
 F 3 "~" H 4050 4500 50  0001 C CNN
 	1    4050 4500
