File: trabajoProfesional/Bateria.sch (KiCad schematic (older format))
At the start: 28 parts, among them T1 MPMOS

Commit message: se agregan los nuevos tamanios de componentes
Parts:
- removed T1: MPMOS, Package_TO_SOT_SMD:TSOT-23, symbol pspice:MPMOS
- added Q1: BSS84, BSS84:SOT95P240X120-3N, symbol BSS84:BSS84
- Cbat1, Cbst1, Cin1, Cin2, Cout1, Cout2, Cout3, Cout4, Cvin1: footprint Capacitor_SMD:C_0201_0603Metric -> Capacitor_SMD:C_0805_2012Metric
- R1fb1, R2fb1, RIPRGM1, Riso_pd1, Rmod_cfg1, Rstatus1: footprint Resistor_SMD:R_0201_0603Metric -> Resistor_SMD:R_0805_2012Metric
Connections:
- wire segments 125 -> 126
Changed lines of the file:
@@
 EESchema Schematic File Version 4
-LIBS:trabajoProfesional-cache
-EELAYER 26 0
+EELAYER 30 0
 EELAYER END
 $Descr A4 11693 8268
@@
 F 0 "Cbst1" H 2185 3004 50  0000 R CNN
 F 1 "47n" H 2185 3095 50  0000 R CNN
-F 2 "Capacitor_SMD:C_0201_0603Metric" H 2338 2900 50  0001 C CNN
+F 2 "Capacitor_SMD:C_0805_2012Metric" H 2338 2900 50  0001 C CNN
 F 3 "~" H 2300 3050 50  0001 C CNN
 	1    2300 3050
@@
 F 0 "Cin1" H 5185 2304 50  0000 R CNN
 F 1 "22u" H 5185 2395 50  0000 R CNN
-F 2 "Capacitor_SMD:C_0201_0603Metric" H 5338 2200 50  0001 C CNN
+F 2 "Capacitor_SMD:C_0805_2012Metric" H 5338 2200 50  0001 C CNN
 F 3 "~" H 5300 2350 50  0001 C CNN
 	1    5300 2350
@@
 F 0 "Rmod_cfg1" H 5620 2946 50  0000 L CNN
 F 1 "60k" H 5620 2855 50  0000 L CNN
-F 2 "Resistor_SMD:R_0201_0603Metric" V 5480 2900 50  0001 C CNN
+F 2 "Resistor_SMD:R_0805_2012Metric" V 5480 2900 50  0001 C CNN
 F 3 "~" H 5550 2900 50  0001 C CNN
 	1    5550 2900
@@
 F 0 "Cin2" H 5585 2304 50  0000 R CNN
 F 1 "100n" H 5585 2395 50  0000 R CNN
-F 2 "Capacitor_SMD:C_0201_0603Metric" H 5738 2200 50  0001 C CNN
+F 2 "Capacitor_SMD:C_0805_2012Metric" H 5738 2200 50  0001 C CNN
 F 3 "~" H 5700 2350 50  0001 C CNN
 	1    5700 2350
@@
 F 0 "R1fb1" H 7370 2696 50  0000 L CNN
 F 1 "46k" H 7370 2605 50  0000 L CNN
-F 2 "Resistor_SMD:R_0201_0603Metric" V 7230 2650 50  0001 C CNN
+F 2 "Resistor_SMD:R_0805_2012Metric" V 7230 2650 50  0001 C CNN
 F 3 "~" H 7300 2650 50  0001 C CNN
 	1    7300 2650
@@
 F 0 "R2fb1" H 7230 3004 50  0000 R CNN
 F 1 "10k" H 7230 3095 50  0000 R CNN
-F 2 "Resistor_SMD:R_0201_0603Metric" V 7230 3050 50  0001 C CNN
+F 2 "Resistor_SMD:R_0805_2012Metric" V 7230 3050 50  0001 C CNN
 F 3 "~" H 7300 3050 50  0001 C CNN
 	1    7300 3050
@@
 F 0 "Cout1" H 7535 2604 50  0000 R CNN
 F 1 "22u" H 7535 2695 50  0000 R CNN
-F 2 "Capacitor_SMD:C_0201_0603Metric" H 7688 2500 50  0001 C CNN
+F 2 "Capacitor_SMD:C_0805_2012Metric" H 7688 2500 50  0001 C CNN
 F 3 "~" H 7650 2650 50  0001 C CNN
 	1    7650 2650
@@
 F 0 "Cout2" H 7935 2604 50  0000 R CNN
 F 1 "22u" H 7935 2695 50  0000 R CNN
-F 2 "Capacitor_SMD:C_0201_0603Metric" H 8088 2500 50  0001 C CNN
+F 2 "Capacitor_SMD:C_0805_2012Metric" H 8088 2500 50  0001 C CNN
 F 3 "~" H 8050 2650 50  0001 C CNN
 	1    8050 2650
@@
 F 0 "Cout3" H 8335 2604 50  0000 R CNN
 F 1 "22u" H 8335 2695 50  0000 R CNN
-F 2 "Capacitor_SMD:C_0201_0603Metric" H 8488 2500 50  0001 C CNN
+F 2 "Capacitor_SMD:C_0805_2012Metric" H 8488 2500 50  0001 C CNN
 F 3 "~" H 8450 2650 50  0001 C CNN
 	1    8450 2650
@@
 F 0 "Cout4" H 8635 2604 50  0000 R CNN
 F 1 "22u" H 8635 2695 50  0000 R CNN
-F 2 "Capacitor_SMD:C_0201_0603Metric" H 8788 2500 50  0001 C CNN
+F 2 "Capacitor_SMD:C_0805_2012Metric" H 8788 2500 50  0001 C CNN
 F 3 "~" H 8750 2650 50  0001 C CNN
 	1    8750 2650
@@
 F 0 "RIPRGM1" V 4893 5200 50  0000 C CNN
 F 1 "10k" V 4984 5200 50  0000 C CNN
-F 2 "Resistor_SMD:R_0201_0603Metric" V 5030 5200 50  0001 C CNN
+F 2 "Resistor_SMD:R_0805_2012Metric" V 5030 5200 50  0001 C CNN
 F 3 "~" H 5100 5200 50  0001 C CNN
 	1    5100 5200
@@
 F 0 "Cbat1" H 6265 5296 50  0000 L CNN
 F 1 "2.2u" H 6265 5205 50  0000 L CNN
-F 2 "Capacitor_SMD:C_0201_0603Metric" H 6188 5100 50  0001 C CNN
+F 2 "Capacitor_SMD:C_0805_2012Metric" H 6188 5100 50  0001 C CNN
 F 3 "~" H 6150 5250 50  0001 C CNN
 	1    6150 5250
@@
 +Bat
 Wire Wire Line
-	7300 5050 6150 5050
+	7300 5050 7200 5050
 Connection ~ 6150 5050
-$Comp
-L pspice:MPMOS T1
-U 1 1 5F4412C3
-P 7200 4750
-F 0 "T1" H 7488 4796 50  0000 L CNN
-F 1 "MPMOS" H 7488 4705 50  0000 L CNN
-F 2 "Package_TO_SOT_SMD:TSOT-23" H 7200 4750 50  0001 C CNN
-F 3 "~" H 7200 4750 50  0001 C CNN
-	1    7200 4750
-	1    0    0    -1
-$EndComp
-Wire Wire Line
-	7400 4550 7300 4550
-Wire Wire Line
-	7300 4950 7300 5050
-Connection ~ 7300 5050
 Text HLabel 9100 4450 2    50   Input ~ 0
 AlimentacionCircuito
@@
 Wire Wire Line
 	7950 4450 7950 4050
-Wire Wire Line
-	7950 4050 7300 4050
-Wire Wire Line
-	7300 4050 7300 4550
-Connection ~ 7300 4550
 $Comp
 L Device:R Riso_pd1
@@
 F 0 "Riso_pd1" H 6330 4654 50  0000 R CNN
 F 1 "R" H 6330 4745 50  0000 R CNN
-F 2 "Resistor_SMD:R_0201_0603Metric" V 6330 4700 50  0001 C CNN
+F 2 "Resistor_SMD:R_0805_2012Metric" V 6330 4700 50  0001 C CNN
 F 3 "~" H 6400 4700 50  0001 C CNN
 	1    6400 4700
@@
 $EndComp
 Wire Wire Line
-	7000 4750 7000 4550
-Wire Wire Line
-	7000 4550 6400 4550
-Wire Wire Line
 	6400 4850 6400 5400
 Wire Wire Line
@@
 	6150 5400 6400 5400
 Wire Wire Line
-	6400 4550 6400 3700
+	6400 4550 6400 4400
 Wire Wire Line
 	3500 3700 6400 3700
-Connection ~ 6400 4550
 Connection ~ 6400 3700
 Wire Wire Line
@@
 F 0 "Cvin1" V 2848 4750 50  0000 C CNN
 F 1 "2.2u" V 2939 4750 50  0000 C CNN
-F 2 "Capacitor_SMD:C_0201_0603Metric" H 3138 4600 50  0001 C CNN
+F 2 "Capacitor_SMD:C_0805_2012Metric" H 3138 4600 50  0001 C CNN
 F 3 "~" H 3100 4750 50  0001 C CNN
 	1    3100 4750
@@
 	5700 4450 5700 4050
 Wire Wire Line
-	5700 4050 7300 4050
-Connection ~ 7300 4050
+	5700 4050 7200 4050
 Wire Wire Line
 	5450 4050 5700 4050
@@
 F 0 "Rstatus1" V 3843 4500 50  0000 C CNN
 F 1 "10k" V 3934 4500 50  0000 C CNN
-F 2 "Resistor_SMD:R_0201_0603Metric" V 3980 4500 50  0001 C CNN
+F 2 "Resistor_SMD:R_0805_2012Metric" V 3980 4500 50  0001 C CNN
 F 3 "~" H 4050 4500 50  0001 C CNN
 	1    4050 4500
@@
 Wire Wire Line
 	5150 2200 5300 2200
+$Comp
+L BSS84:BSS84 Q1
+U 1 1 5FB6037E
+P 6900 4600
+F 0 "Q1" H 7330 4654 50  0000 L CNN
+F 1 "BSS84" H 7330 4745 50  0000 L CNN
+F 2 "BSS84:SOT95P240X120-3N" H 7350 4550 50  0001 L CNN
+F 3 "http://www.onsemi.com/pub/Collateral/BSS84-D.PDF" H 7350 4450 50  0001 L CNN
+F 4 "P-Channel Enhancement Mode Field Effect Transistor" H 7350 4350 50  0001 L CNN "Description"
+F 5 "1.2" H 7350 4250 50  0001 L CNN "Height"
+F 6 "512-BSS84" H 7350 4150 50  0001 L CNN "Mouser Part Number"
+F 7 "https://www.mouser.co.uk/ProductDetail/ON-Semiconductor-Fairchild/BSS84?qs=FOlmdCx%252BAA0e83h5MpSc0g%3D%3D" H 7350 4050 50  0001 L CNN "Mouser Price/Stock"
+F 8 "ON Semiconductor" H 7350 3950 50  0001 L CNN "Manufacturer_Name"
+F 9 "BSS84" H 7350 3850 50  0001 L CNN "Manufacturer_Part_Number"
+	1    6900 4600
+	1    0    0    1
+$EndComp
+Wire Wire Line
+	7200 4400 7200 4050
+Connection ~ 7200 4050
+Wire Wire Line
+	7200 4050 7950 4050
+Wire Wire Line
+	6900 4600 6900 4400
+Wire Wire Line
+	6900 4400 6400 4400
+Connection ~ 6400 4400
+Wire Wire Line
+	6400 4400 6400 3700
+Wire Wire Line
+	7200 5000 7200 5050
+Connection ~ 7200 5050
+Wire Wire Line
+	7200 5050 6150 5050
 $EndSCHEMATC
