File: trabajoProfesional/Bateria.sch (KiCad schematic (older format))
At the start: 28 parts, among them Q1 BSS84

Commit message: Revert "Ultimas modificaciones de las lineas"
se vuelve al estado anterior!

This reverts commit 6775e72ca7e72ceb68c45e191fec203a9774ccb5.
Parts:
- Q1: symbol trabajoProfesional-rescue:BSS84-BSS84 -> BSS84:BSS84
Changed lines of the file:
@@
 EESchema Schematic File Version 4
-LIBS:trabajoProfesional-cache
-EELAYER 26 0
+EELAYER 30 0
 EELAYER END
 $Descr A4 11693 8268
@@
 	5150 2200 5300 2200
 $Comp
-L trabajoProfesional-rescue:BSS84-BSS84 Q1
+L BSS84:BSS84 Q1
 U 1 1 5FB6037E
 P 6900 4600
