File: trabajoProfesional/salida.sch (KiCad schematic (older format))
At the start: 11 parts

Commit message: ya tenemos los componentes falta el micro
Parts:
- C1, C2, C3, C4, C5: value C -> 10n
- D1, D2, D3, D4: value D -> 1.8
Connections:
- net VLL renamed Alimentacion
Changed lines of the file:
@@
 AR Path="/5F3D0683/5F3DE12E" Ref="D1"  Part="1"
 F 0 "D1" H 7550 2767 50  0000 C CNN
-F 1 "D" H 7550 2676 50  0000 C CNN
+F 1 "1.8" H 7550 2676 50  0000 C CNN
 F 2 "" H 7550 2550 50  0001 C CNN
 F 3 "~" H 7550 2550 50  0001 C CNN
@@
 AR Path="/5F3D0683/5F3DE134" Ref="D2"  Part="1"
 F 0 "D2" H 7250 2133 50  0000 C CNN
-F 1 "D" H 7250 2224 50  0000 C CNN
+F 1 "1.8" H 7250 2224 50  0000 C CNN
 F 2 "" H 7250 2350 50  0001 C CNN
 F 3 "~" H 7250 2350 50  0001 C CNN
@@
 AR Path="/5F3D0683/5F3DE13A" Ref="D4"  Part="1"
 F 0 "D4" H 7300 1633 50  0000 C CNN
-F 1 "D" H 7300 1724 50  0000 C CNN
+F 1 "1.8" H 7300 1724 50  0000 C CNN
 F 2 "" H 7300 1850 50  0001 C CNN
 F 3 "~" H 7300 1850 50  0001 C CNN
@@
 AR Path="/5F3D0683/5F3DE140" Ref="D3"  Part="1"
 F 0 "D3" H 7550 2267 50  0000 C CNN
-F 1 "D" H 7550 2176 50  0000 C CNN
+F 1 "1.8" H 7550 2176 50  0000 C CNN
 F 2 "" H 7550 2050 50  0001 C CNN
 F 3 "~" H 7550 2050 50  0001 C CNN
@@
 Wire Wire Line
 	2350 1200 2350 2600
-Text GLabel 2350 1200 0    50   Input ~ 0
-VLL
 Connection ~ 5850 1200
 Connection ~ 6600 1650
@@
 AR Path="/5F3D0683/5F3DE174" Ref="C3"  Part="1"
 F 0 "C3" V 4298 3000 50  0000 C CNN
-F 1 "C" V 4389 3000 50  0000 C CNN
+F 1 "10n" V 4389 3000 50  0000 C CNN
 F 2 "" H 4588 2850 50  0001 C CNN
 F 3 "~" H 4550 3000 50  0001 C CNN
 	1    4550 3000
-	0    1    1    0
-$EndComp
-$Comp
-L Device:C C?
-U 1 1 5F3DE17A
-P 3650 2050
-AR Path="/5F3DE17A" Ref="C?"  Part="1"
-AR Path="/5F3D0683/5F3DE17A" Ref="C1"  Part="1"
-F 0 "C1" V 3398 2050 50  0000 C CNN
-F 1 "C" V 3489 2050 50  0000 C CNN
-F 2 "" H 3688 1900 50  0001 C CNN
-F 3 "~" H 3650 2050 50  0001 C CNN
-	1    3650 2050
 	0    1    1    0
 $EndComp
@@
 AR Path="/5F3D0683/5F3DE180" Ref="C4"  Part="1"
 F 0 "C4" V 6198 2650 50  0000 C CNN
-F 1 "C" V 6289 2650 50  0000 C CNN
+F 1 "10n" V 6289 2650 50  0000 C CNN
 F 2 "" H 6488 2500 50  0001 C CNN
 F 3 "~" H 6450 2650 50  0001 C CNN
@@
 AR Path="/5F3D0683/5F3DE186" Ref="C5"  Part="1"
 F 0 "C5" V 5948 2350 50  0000 C CNN
-F 1 "C" V 6039 2350 50  0000 C CNN
+F 1 "10n" V 6039 2350 50  0000 C CNN
 F 2 "" H 6238 2200 50  0001 C CNN
 F 3 "~" H 6200 2350 50  0001 C CNN
@@
 AR Path="/5F3D0683/5F3DE18C" Ref="C2"  Part="1"
 F 0 "C2" V 3198 2350 50  0000 C CNN
-F 1 "C" V 3289 2350 50  0000 C CNN
+F 1 "10n" V 3289 2350 50  0000 C CNN
 F 2 "" H 3488 2200 50  0001 C CNN
 F 3 "~" H 3450 2350 50  0001 C CNN
@@
 Wire Wire Line
 	1500 3100 4050 3100
+Text HLabel 2050 1200 0    50   Input ~ 0
+Alimentacion
+Wire Wire Line
+	2050 1200 2350 1200
+$Comp
+L Device:C C?
+U 1 1 5F3DE17A
+P 3650 2050
+AR Path="/5F3DE17A" Ref="C?"  Part="1"
+AR Path="/5F3D0683/5F3DE17A" Ref="C1"  Part="1"
+F 0 "C1" V 3398 2050 50  0000 C CNN
+F 1 "10n" V 3489 2050 50  0000 C CNN
+F 2 "" H 3688 1900 50  0001 C CNN
+F 3 "~" H 3650 2050 50  0001 C CNN
+	1    3650 2050
+	0    1    1    0
+$EndComp
 $EndSCHEMATC

Commit message: empezando el pcb
Parts:
- C1, C2, C3, C4, C5: footprint (none) -> Capacitor_SMD:C_2816_7142Metric
- D1, D2, D3, D4: footprint (none) -> Diode_SMD:D_SC-80
- DriverPotencia1: renamed from DriverPotencia; footprint HV7360GAG -> HV7360:HV7360GAG
- PiezoElectrico1: renamed from PiezoElectrico; footprint UTR1440KTTR -> Connector_PinHeader_2.54mm:PinHeader_1x02_P2.54mm_Vertical
Changed lines of the file:
@@
 P 8950 2100
 AR Path="/5F3DE108" Ref="PiezoElectrico?"  Part="1"
-AR Path="/5F3D0683/5F3DE108" Ref="PiezoElectrico"  Part="1"
-F 0 "PiezoElectrico" H 9578 2096 50  0000 L CNN
+AR Path="/5F3D0683/5F3DE108" Ref="PiezoElectrico1"  Part="1"
+F 0 "PiezoElectrico1" H 9578 2096 50  0000 L CNN
 F 1 "UTR-1440K-TT-R" H 9578 2005 50  0000 L CNN
-F 2 "UTR1440KTTR" H 9600 2200 50  0001 L CNN
+F 2 "Connector_PinHeader_2.54mm:PinHeader_1x02_P2.54mm_Vertical" H 9600 2200 50  0001 L CNN
 F 3 "http://www.puiaudio.com/pdf/UTR-1440K-TT-R.pdf" H 9600 2100 50  0001 L CNN
 F 4 "Speakers & Transducers ULTRASONIC TRNSMTTR /RECEIVER" H 9600 2000 50  0001 L CNN "Description"
@@
 F 0 "D1" H 7550 2767 50  0000 C CNN
 F 1 "1.8" H 7550 2676 50  0000 C CNN
-F 2 "" H 7550 2550 50  0001 C CNN
+F 2 "Diode_SMD:D_SC-80" H 7550 2550 50  0001 C CNN
 F 3 "~" H 7550 2550 50  0001 C CNN
 	1    7550 2550
@@
 F 0 "D2" H 7250 2133 50  0000 C CNN
 F 1 "1.8" H 7250 2224 50  0000 C CNN
-F 2 "" H 7250 2350 50  0001 C CNN
+F 2 "Diode_SMD:D_SC-80" H 7250 2350 50  0001 C CNN
 F 3 "~" H 7250 2350 50  0001 C CNN
 	1    7250 2350
@@
 F 0 "D4" H 7300 1633 50  0000 C CNN
 F 1 "1.8" H 7300 1724 50  0000 C CNN
-F 2 "" H 7300 1850 50  0001 C CNN
+F 2 "Diode_SMD:D_SC-80" H 7300 1850 50  0001 C CNN
 F 3 "~" H 7300 1850 50  0001 C CNN
 	1    7300 1850
@@
 F 0 "D3" H 7550 2267 50  0000 C CNN
 F 1 "1.8" H 7550 2176 50  0000 C CNN
-F 2 "" H 7550 2050 50  0001 C CNN
+F 2 "Diode_SMD:D_SC-80" H 7550 2050 50  0001 C CNN
 F 3 "~" H 7550 2050 50  0001 C CNN
 	1    7550 2050
@@
 F 0 "C3" V 4298 3000 50  0000 C CNN
 F 1 "10n" V 4389 3000 50  0000 C CNN
-F 2 "" H 4588 2850 50  0001 C CNN
+F 2 "Capacitor_SMD:C_2816_7142Metric" H 4588 2850 50  0001 C CNN
 F 3 "~" H 4550 3000 50  0001 C CNN
 	1    4550 3000
@@
 F 0 "C4" V 6198 2650 50  0000 C CNN
 F 1 "10n" V 6289 2650 50  0000 C CNN
-F 2 "" H 6488 2500 50  0001 C CNN
+F 2 "Capacitor_SMD:C_2816_7142Metric" H 6488 2500 50  0001 C CNN
 F 3 "~" H 6450 2650 50  0001 C CNN
 	1    6450 2650
@@
 F 0 "C5" V 5948 2350 50  0000 C CNN
 F 1 "10n" V 6039 2350 50  0000 C CNN
-F 2 "" H 6238 2200 50  0001 C CNN
+F 2 "Capacitor_SMD:C_2816_7142Metric" H 6238 2200 50  0001 C CNN
 F 3 "~" H 6200 2350 50  0001 C CNN
 	1    6200 2350
@@
 F 0 "C2" V 3198 2350 50  0000 C CNN
 F 1 "10n" V 3289 2350 50  0000 C CNN
-F 2 "" H 3488 2200 50  0001 C CNN
+F 2 "Capacitor_SMD:C_2816_7142Metric" H 3488 2200 50  0001 C CNN
 F 3 "~" H 3450 2350 50  0001 C CNN
 	1    3450 2350
@@
 P 3900 1550
 AR Path="/5F3DE1A4" Ref="#PWR?"  Part="1"
-AR Path="/5F3D0683/5F3DE1A4" Ref="#PWR?"  Part="1"
-F 0 "#PWR?" H 3900 1300 50  0001 C CNN
+AR Path="/5F3D0683/5F3DE1A4" Ref="#PWR0102"  Part="1"
+F 0 "#PWR0102" H 3900 1300 50  0001 C CNN
 F 1 "GND" H 3905 1377 50  0000 C CNN
 F 2 "" H 3900 1550 50  0001 C CNN
@@
 P 4500 1650
 AR Path="/5F3DE1B0" Ref="DriverPotencia?"  Part="1"
-AR Path="/5F3D0683/5F3DE1B0" Ref="DriverPotencia"  Part="1"
-F 0 "DriverPotencia" H 5050 1915 50  0000 C CNN
+AR Path="/5F3D0683/5F3DE1B0" Ref="DriverPotencia1"  Part="1"
+F 0 "DriverPotencia1" H 5050 1915 50  0000 C CNN
 F 1 "HV7360GA-G" H 5050 1824 50  0000 C CNN
-F 2 "HV7360GAG" H 5450 1750 50  0001 L CNN
+F 2 "HV7360:HV7360GAG" H 5450 1750 50  0001 L CNN
 F 3 "http://www.microchip.com/mymicrochip/filehandler.aspx?ddocname=en571410" H 5450 1650 50  0001 L CNN
 F 4 "Power Management Specialized - PMIC 1-Ch +/-100V 2.5A 2/3-Lev AC Coupled Pulser" H 5450 1550 50  0001 L CNN "Description"
@@
 F 0 "C1" V 3398 2050 50  0000 C CNN
 F 1 "10n" V 3489 2050 50  0000 C CNN
-F 2 "" H 3688 1900 50  0001 C CNN
+F 2 "Capacitor_SMD:C_2816_7142Metric" H 3688 1900 50  0001 C CNN
 F 3 "~" H 3650 2050 50  0001 C CNN
 	1    3650 2050

Commit message: paso previo PCB
Parts:
- added 10V1: Conn_01x01_Male, Connector_PinHeader_1.00mm:PinHeader_1x01_P1.00mm_Vertical, symbol Connector:Conn_01x01_Male
- added HV+1, HV-1: Conn_01x01_Male, Connector_PinSocket_2.54mm:PinSocket_1x01_P2.54mm_Vertical, symbol Connector:Conn_01x01_Male
Connections:
- net +HV: now also HV+1.1 (Pin_1)
- net -HV: now also HV-1.1 (Pin_1)
- net 10V: now also 10V1.1 (Pin_1)
Changed lines of the file:
@@
 	4000 2050 4500 2050
 Connection ~ 4000 2050
-Wire Wire Line
-	4000 1850 4000 2050
 Text GLabel 4000 1850 0    50   Input ~ 0
 10V
@@
 Connection ~ 6250 2650
 Wire Wire Line
-	6250 3250 6250 2650
+	6250 3250 6250 3200
 Text GLabel 6250 3250 2    50   Input ~ 0
 -HV
@@
 Wire Wire Line
 	4500 2550 4200 2550
-Wire Wire Line
-	4200 1550 3900 1550
 Connection ~ 4200 1550
 Wire Wire Line
@@
 	4500 1950 4200 1950
 Wire Wire Line
-	4400 1550 4200 1550
+	4400 1550 4300 1550
 Wire Wire Line
 	4400 1650 4400 1550
@@
 L power:GND #PWR?
 U 1 1 5F3DE1A4
-P 3900 1550
+P 4300 1550
 AR Path="/5F3DE1A4" Ref="#PWR?"  Part="1"
 AR Path="/5F3D0683/5F3DE1A4" Ref="#PWR0102"  Part="1"
-F 0 "#PWR0102" H 3900 1300 50  0001 C CNN
-F 1 "GND" H 3905 1377 50  0000 C CNN
-F 2 "" H 3900 1550 50  0001 C CNN
-F 3 "" H 3900 1550 50  0001 C CNN
-	1    3900 1550
+F 0 "#PWR0102" H 4300 1300 50  0001 C CNN
+F 1 "GND" H 4305 1377 50  0000 C CNN
+F 2 "" H 4300 1550 50  0001 C CNN
+F 3 "" H 4300 1550 50  0001 C CNN
+	1    4300 1550
 	1    0    0    -1
 $EndComp
@@
 	0    1    1    0
 $EndComp
+Wire Wire Line
+	5950 3600 5950 3250
+Wire Wire Line
+	5950 3250 5850 3250
+Connection ~ 5850 3250
+Wire Wire Line
+	6250 3200 6050 3200
+Wire Wire Line
+	6050 3200 6050 3700
+Connection ~ 6250 3200
+Wire Wire Line
+	6250 3200 6250 2650
+$Comp
+L Connector:Conn_01x01_Male 10V1
+U 1 1 5F407A63
+P 3650 1450
+F 0 "10V1" H 3758 1631 50  0000 C CNN
+F 1 "Conn_01x01_Male" H 3758 1540 50  0000 C CNN
+F 2 "Connector_PinHeader_1.00mm:PinHeader_1x01_P1.00mm_Vertical" H 3650 1450 50  0001 C CNN
+F 3 "~" H 3650 1450 50  0001 C CNN
+	1    3650 1450
+	1    0    0    -1
+$EndComp
+Wire Wire Line
+	4000 1450 3850 1450
+Wire Wire Line
+	4000 1450 4000 2050
+Connection ~ 4300 1550
+Wire Wire Line
+	4300 1550 4200 1550
+$Comp
+L Connector:Conn_01x01_Male HV+1
+U 1 1 5F42DBC3
+P 5350 3600
+F 0 "HV+1" H 5458 3781 50  0000 C CNN
+F 1 "Conn_01x01_Male" H 5458 3690 50  0000 C CNN
+F 2 "Connector_PinSocket_2.54mm:PinSocket_1x01_P2.54mm_Vertical" H 5350 3600 50  0001 C CNN
+F 3 "~" H 5350 3600 50  0001 C CNN
+	1    5350 3600
+	1    0    0    -1
+$EndComp
+$Comp
+L Connector:Conn_01x01_Male HV-1
+U 1 1 5F42E43A
+P 6500 3700
+F 0 "HV-1" H 6472 3632 50  0000 R CNN
+F 1 "Conn_01x01_Male" H 6472 3723 50  0000 R CNN
+F 2 "Connector_PinSocket_2.54mm:PinSocket_1x01_P2.54mm_Vertical" H 6500 3700 50  0001 C CNN
+F 3 "~" H 6500 3700 50  0001 C CNN
+	1    6500 3700
+	-1   0    0    1
+$EndComp
+Wire Wire Line
+	5950 3600 5550 3600
+Wire Wire Line
+	6300 3700 6050 3700
 $EndSCHEMATC

Commit message: PCB falta una conexion
Parts:
- 10V1: footprint Connector_PinHeader_1.00mm:PinHeader_1x01_P1.00mm_Vertical -> TestPoint:TestPoint_Pad_D2.5mm
- HV+1, HV-1: footprint Connector_PinSocket_2.54mm:PinSocket_1x01_P2.54mm_Vertical -> TestPoint:TestPoint_Pad_D2.5mm
- PiezoElectrico1: footprint Connector_PinHeader_2.54mm:PinHeader_1x02_P2.54mm_Vertical -> Connector_PinHeader_2.54mm:PinHeader_1x02_P2.54mm_Vertical_SMD_Pin1Left
Changed lines of the file:
@@
 F 0 "PiezoElectrico1" H 9578 2096 50  0000 L CNN
 F 1 "UTR-1440K-TT-R" H 9578 2005 50  0000 L CNN
-F 2 "Connector_PinHeader_2.54mm:PinHeader_1x02_P2.54mm_Vertical" H 9600 2200 50  0001 L CNN
+F 2 "Connector_PinHeader_2.54mm:PinHeader_1x02_P2.54mm_Vertical_SMD_Pin1Left" H 9600 2200 50  0001 L CNN
 F 3 "http://www.puiaudio.com/pdf/UTR-1440K-TT-R.pdf" H 9600 2100 50  0001 L CNN
 F 4 "Speakers & Transducers ULTRASONIC TRNSMTTR /RECEIVER" H 9600 2000 50  0001 L CNN "Description"
@@
 F 0 "10V1" H 3758 1631 50  0000 C CNN
 F 1 "Conn_01x01_Male" H 3758 1540 50  0000 C CNN
-F 2 "Connector_PinHeader_1.00mm:PinHeader_1x01_P1.00mm_Vertical" H 3650 1450 50  0001 C CNN
+F 2 "TestPoint:TestPoint_Pad_D2.5mm" H 3650 1450 50  0001 C CNN
 F 3 "~" H 3650 1450 50  0001 C CNN
 	1    3650 1450
@@
 F 0 "HV+1" H 5458 3781 50  0000 C CNN
 F 1 "Conn_01x01_Male" H 5458 3690 50  0000 C CNN
-F 2 "Connector_PinSocket_2.54mm:PinSocket_1x01_P2.54mm_Vertical" H 5350 3600 50  0001 C CNN
+F 2 "TestPoint:TestPoint_Pad_D2.5mm" H 5350 3600 50  0001 C CNN
 F 3 "~" H 5350 3600 50  0001 C CNN
 	1    5350 3600
@@
 F 0 "HV-1" H 6472 3632 50  0000 R CNN
 F 1 "Conn_01x01_Male" H 6472 3723 50  0000 R CNN
-F 2 "Connector_PinSocket_2.54mm:PinSocket_1x01_P2.54mm_Vertical" H 6500 3700 50  0001 C CNN
+F 2 "TestPoint:TestPoint_Pad_D2.5mm" H 6500 3700 50  0001 C CNN
 F 3 "~" H 6500 3700 50  0001 C CNN
 	1    6500 3700

Commit message: va el circuito
Parts:
- C1, C2, C3, C4, C5: footprint Capacitor_SMD:C_2816_7142Metric -> Capacitor_SMD:C_0201_0603Metric
Changed lines of the file:
@@
 F 0 "C3" V 4298 3000 50  0000 C CNN
 F 1 "10n" V 4389 3000 50  0000 C CNN
-F 2 "Capacitor_SMD:C_2816_7142Metric" H 4588 2850 50  0001 C CNN
+F 2 "Capacitor_SMD:C_0201_0603Metric" H 4588 2850 50  0001 C CNN
 F 3 "~" H 4550 3000 50  0001 C CNN
 	1    4550 3000
@@
 F 0 "C4" V 6198 2650 50  0000 C CNN
 F 1 "10n" V 6289 2650 50  0000 C CNN
-F 2 "Capacitor_SMD:C_2816_7142Metric" H 6488 2500 50  0001 C CNN
+F 2 "Capacitor_SMD:C_0201_0603Metric" H 6488 2500 50  0001 C CNN
 F 3 "~" H 6450 2650 50  0001 C CNN
 	1    6450 2650
@@
 F 0 "C5" V 5948 2350 50  0000 C CNN
 F 1 "10n" V 6039 2350 50  0000 C CNN
-F 2 "Capacitor_SMD:C_2816_7142Metric" H 6238 2200 50  0001 C CNN
+F 2 "Capacitor_SMD:C_0201_0603Metric" H 6238 2200 50  0001 C CNN
 F 3 "~" H 6200 2350 50  0001 C CNN
 	1    6200 2350
@@
 F 0 "C2" V 3198 2350 50  0000 C CNN
 F 1 "10n" V 3289 2350 50  0000 C CNN
-F 2 "Capacitor_SMD:C_2816_7142Metric" H 3488 2200 50  0001 C CNN
+F 2 "Capacitor_SMD:C_0201_0603Metric" H 3488 2200 50  0001 C CNN
 F 3 "~" H 3450 2350 50  0001 C CNN
 	1    3450 2350
@@
 F 0 "C1" V 3398 2050 50  0000 C CNN
 F 1 "10n" V 3489 2050 50  0000 C CNN
-F 2 "Capacitor_SMD:C_2816_7142Metric" H 3688 1900 50  0001 C CNN
+F 2 "Capacitor_SMD:C_0201_0603Metric" H 3688 1900 50  0001 C CNN
 F 3 "~" H 3650 2050 50  0001 C CNN
 	1    3650 2050

Commit message: va lo actual
Parts:
- C1, C2, C3, C5: value 10n -> 4.7u
- C4: value 10n -> 4.7
Changed lines of the file:
@@
 AR Path="/5F3D0683/5F3DE174" Ref="C3"  Part="1"
 F 0 "C3" V 4298 3000 50  0000 C CNN
-F 1 "10n" V 4389 3000 50  0000 C CNN
+F 1 "4.7u" V 4389 3000 50  0000 C CNN
 F 2 "Capacitor_SMD:C_0201_0603Metric" H 4588 2850 50  0001 C CNN
 F 3 "~" H 4550 3000 50  0001 C CNN
@@
 AR Path="/5F3D0683/5F3DE180" Ref="C4"  Part="1"
 F 0 "C4" V 6198 2650 50  0000 C CNN
-F 1 "10n" V 6289 2650 50  0000 C CNN
+F 1 "4.7" V 6289 2650 50  0000 C CNN
 F 2 "Capacitor_SMD:C_0201_0603Metric" H 6488 2500 50  0001 C CNN
 F 3 "~" H 6450 2650 50  0001 C CNN
@@
 AR Path="/5F3D0683/5F3DE186" Ref="C5"  Part="1"
 F 0 "C5" V 5948 2350 50  0000 C CNN
-F 1 "10n" V 6039 2350 50  0000 C CNN
+F 1 "4.7u" V 6039 2350 50  0000 C CNN
 F 2 "Capacitor_SMD:C_0201_0603Metric" H 6238 2200 50  0001 C CNN
 F 3 "~" H 6200 2350 50  0001 C CNN
@@
 AR Path="/5F3D0683/5F3DE18C" Ref="C2"  Part="1"
 F 0 "C2" V 3198 2350 50  0000 C CNN
-F 1 "10n" V 3289 2350 50  0000 C CNN
+F 1 "4.7u" V 3289 2350 50  0000 C CNN
 F 2 "Capacitor_SMD:C_0201_0603Metric" H 3488 2200 50  0001 C CNN
 F 3 "~" H 3450 2350 50  0001 C CNN
@@
 AR Path="/5F3D0683/5F3DE17A" Ref="C1"  Part="1"
 F 0 "C1" V 3398 2050 50  0000 C CNN
-F 1 "10n" V 3489 2050 50  0000 C CNN
+F 1 "4.7u" V 3489 2050 50  0000 C CNN
 F 2 "Capacitor_SMD:C_0201_0603Metric" H 3688 1900 50  0001 C CNN
 F 3 "~" H 3650 2050 50  0001 C CNN

Commit message: Add files via upload
Parts:
- D1, D2, D3, D4: footprint Diode_SMD:D_SC-80 -> Diode_SMD:D_SOD-123
- DriverPotencia1: symbol HV7360GA-G:HV7360GA-G -> trabajoProfesional-rescue:HV7360GA-G-HV7360GA-G
- PiezoElectrico1: symbol UTR-1440K-TT-R:UTR-1440K-TT-R -> trabajoProfesional-rescue:UTR-1440K-TT-R-UTR-1440K-TT-R
Changed lines of the file:
@@
 EESchema Schematic File Version 4
-EELAYER 30 0
+LIBS:trabajoProfesional-cache
+EELAYER 26 0
 EELAYER END
 $Descr A4 11693 8268
@@
 	8950 2200 8250 2200
 $Comp
-L UTR-1440K-TT-R:UTR-1440K-TT-R PiezoElectrico?
+L trabajoProfesional-rescue:UTR-1440K-TT-R-UTR-1440K-TT-R PiezoElectrico?
 U 1 1 5F3DE108
 P 8950 2100
@@
 F 0 "D1" H 7550 2767 50  0000 C CNN
 F 1 "1.8" H 7550 2676 50  0000 C CNN
-F 2 "Diode_SMD:D_SC-80" H 7550 2550 50  0001 C CNN
+F 2 "Diode_SMD:D_SOD-123" H 7550 2550 50  0001 C CNN
 F 3 "~" H 7550 2550 50  0001 C CNN
 	1    7550 2550
@@
 F 0 "D2" H 7250 2133 50  0000 C CNN
 F 1 "1.8" H 7250 2224 50  0000 C CNN
-F 2 "Diode_SMD:D_SC-80" H 7250 2350 50  0001 C CNN
+F 2 "Diode_SMD:D_SOD-123" H 7250 2350 50  0001 C CNN
 F 3 "~" H 7250 2350 50  0001 C CNN
 	1    7250 2350
@@
 F 0 "D4" H 7300 1633 50  0000 C CNN
 F 1 "1.8" H 7300 1724 50  0000 C CNN
-F 2 "Diode_SMD:D_SC-80" H 7300 1850 50  0001 C CNN
+F 2 "Diode_SMD:D_SOD-123" H 7300 1850 50  0001 C CNN
 F 3 "~" H 7300 1850 50  0001 C CNN
 	1    7300 1850
@@
 F 0 "D3" H 7550 2267 50  0000 C CNN
 F 1 "1.8" H 7550 2176 50  0000 C CNN
-F 2 "Diode_SMD:D_SC-80" H 7550 2050 50  0001 C CNN
+F 2 "Diode_SMD:D_SOD-123" H 7550 2050 50  0001 C CNN
 F 3 "~" H 7550 2050 50  0001 C CNN
 	1    7550 2050
@@
 $EndComp
 $Comp
-L HV7360GA-G:HV7360GA-G DriverPotencia?
+L trabajoProfesional-rescue:HV7360GA-G-HV7360GA-G DriverPotencia?
 U 1 1 5F3DE1B0
 P 4500 1650
