File: trabajoProfesional/salida.sch (KiCad schematic (older format))
At the start: 14 parts

Commit message: Ultima placa que imprimimos todo junto
Parts:
- C4: value 4.7 -> 4.7u
Changed lines of the file:
@@
 AR Path="/5F3D0683/5F3DE180" Ref="C4"  Part="1"
 F 0 "C4" V 6198 2650 50  0000 C CNN
-F 1 "4.7" V 6289 2650 50  0000 C CNN
+F 1 "4.7u" V 6289 2650 50  0000 C CNN
 F 2 "Capacitor_SMD:C_0805_2012Metric" H 6488 2500 50  0001 C CNN
 F 3 "~" H 6450 2650 50  0001 C CNN
