File: trabajoProfesional/CargadorBateria.sch (KiCad schematic (older format))
At the start: 30 parts, among them IC1 TS51231-QFNR

Commit message: Revert "Ultimas modificaciones de las lineas"
se vuelve al estado anterior!

This reverts commit 6775e72ca7e72ceb68c45e191fec203a9774ccb5.
Parts:
- IC1: symbol trabajoProfesional-rescue:TS51231-QFNR-TS51231-QFNR -> TS51231-QFNR:TS51231-QFNR
Changed lines of the file:
@@
 EESchema Schematic File Version 4
-LIBS:trabajoProfesional-cache
-EELAYER 26 0
+EELAYER 30 0
 EELAYER END
 $Descr A4 11693 8268
@@
 $EndDescr
 $Comp
-L trabajoProfesional-rescue:TS51231-QFNR-TS51231-QFNR IC1
+L TS51231-QFNR:TS51231-QFNR IC1
 U 1 1 5FFE6889
 P 5400 2900
