File: trabajoProfesional/Centralizador.sch (KiCad schematic (older format))
At the start: 23 parts, among them IC2 HV7361GA-G

Commit message: Revert "Ultimas modificaciones de las lineas"
se vuelve al estado anterior!

This reverts commit 6775e72ca7e72ceb68c45e191fec203a9774ccb5.
Parts:
- D10, D11, D6, D7, D8, D9: symbol trabajoProfesional-rescue:1N4150W-E3-08-Diodo1N4150W-e3-08 -> Diodo1N4150W-e3-08:1N4150W-E3-08
- IC2: symbol trabajoProfesional-rescue:HV7361GA-G-HV7361GA-G -> HV7361GA-G:HV7361GA-G
- LS1: symbol trabajoProfesional-rescue:UTR-1440K-TT-R-UTR-1440K-TT-R -> UTR-1440K-TT-R:UTR-1440K-TT-R
Changed lines of the file:
@@
 EESchema Schematic File Version 4
-LIBS:trabajoProfesional-cache
-EELAYER 26 0
+EELAYER 30 0
 EELAYER END
 $Descr A4 11693 8268
@@
 $EndDescr
 $Comp
-L trabajoProfesional-rescue:HV7361GA-G-HV7361GA-G IC2
+L HV7361GA-G:HV7361GA-G IC2
 U 1 1 5FFE4A75
 P 3900 2200
@@
 $EndComp
 $Comp
-L trabajoProfesional-rescue:UTR-1440K-TT-R-UTR-1440K-TT-R LS1
+L UTR-1440K-TT-R:UTR-1440K-TT-R LS1
 U 1 1 60011CA2
 P 8050 4200
@@
 $EndComp
 $Comp
-L trabajoProfesional-rescue:1N4150W-E3-08-Diodo1N4150W-e3-08 D8
+L Diodo1N4150W-e3-08:1N4150W-E3-08 D8
 U 1 1 60017B33
 P 5850 1800
@@
 $EndComp
 $Comp
-L trabajoProfesional-rescue:1N4150W-E3-08-Diodo1N4150W-e3-08 D9
+L Diodo1N4150W-e3-08:1N4150W-E3-08 D9
 U 1 1 600182E2
 P 6250 2500
@@
 $EndComp
 $Comp
-L trabajoProfesional-rescue:1N4150W-E3-08-Diodo1N4150W-e3-08 D11
+L Diodo1N4150W-e3-08:1N4150W-E3-08 D11
 U 1 1 60018639
 P 6550 2700
@@
 $EndComp
 $Comp
-L trabajoProfesional-rescue:1N4150W-E3-08-Diodo1N4150W-e3-08 D7
+L Diodo1N4150W-e3-08:1N4150W-E3-08 D7
 U 1 1 60018944
 P 5700 4300
@@
 $EndComp
 $Comp
-L trabajoProfesional-rescue:1N4150W-E3-08-Diodo1N4150W-e3-08 D10
+L Diodo1N4150W-e3-08:1N4150W-E3-08 D10
 U 1 1 6001A4A6
 P 6300 3800
@@
 $EndComp
 $Comp
-L trabajoProfesional-rescue:1N4150W-E3-08-Diodo1N4150W-e3-08 D6
+L Diodo1N4150W-e3-08:1N4150W-E3-08 D6
 U 1 1 6001A808
 P 5450 1200
